File: PCB/MixuinoPCB.kicad/MixuinoPCB.kicad_pcb (KiCad board)
At the start: 2 copper layers, 83.8 x 81.3 mm, 13 parts

Commit message: Final commit before merge with main repo, updated KiCAD projects + added the CAD files
Parts:
- turned U1 to 180 degrees
- turned U2 to 180 degrees
- turned U3 to 180 degrees
- turned U4 to 180 degrees
Routing:
- net Net-(A1-A3): track 174.9 -> 31.5 mm
- net Net-(A1-A2): track 148.6 -> 17.9 mm
- net Net-(A1-A1): track 95.0 -> 35.9 mm
- net Net-(A1-A0): track 85.7 -> 43.9 mm
- net Net-(A1-+5V): track 121.2 -> 123.3 mm
- net Net-(A1-GND-Pad29): track 116.1 -> 114.6 mm
Other:
- board text added: "Logo by Inés D'Olha"
- board text added: "github.com/ThePangel"
- board text removed: "Logo: Inés D'Olha"
